Commit message: rviz(r*) launch_Files up

File: pauli/urdf/xacro/model_pauli.xacro (robot description, xacro)
@@ -3,10 +3,10 @@
   <xacro:include filename="$(find pauli)/urdf/xacro/model_pauli_colored.xacro"/>
   <xacro:include filename="$(find pauli)/urdf/xacro/pauli_plugins_gazebo.xacro"/>
-  <!-- <link name="base_footprint"/>
+  <link name="base_footprint"/>
   <joint name="base_joint" type="fixed">
     <parent link="base_footprint"/>
     <child link="base_link"/>
-    <origin xyz="0.0 0.0 0.010" rpy="0 0 0"/>
-  </joint> -->
+    <origin xyz="0.0 0.0 0.0" rpy="0 0 0"/>
+  </joint>
   <link
     name="base_link">
